File: pcb/GPC_dev_board.kicad_pcb (KiCad board)
At the start: 6 copper layers, 182.9 x 100.4 mm, 185 parts, among them J1 Conn_01x12, J10 CTRL, J11 Conn_02x06_Top_Bottom, J12 LVIN, J14 Conn_01x04, J15 Vdc, J16 PWMIN, J17 HBRIDGE, J18 Vac, J19 LVIN, J2 Conn_01x12, J20 LVOUT, J3 Conn_02x13_Odd_Even, J4 Conn_02x13_Odd_Even, J5 BATTERY, J6 SECONDARY, J7 3.3V, Q1 IXFN80N50, Q2 IRF4905, Q3 IRF4905, Q4 IRF4905, Q5 IRF4905, Q6 MMBT3904, Q7 MMBT3904, Q8 MMBT3904, Q9 MMBT3904, U1 AMC3330, U10 ISO7320FC, U11 TLV74325, U12 TLV74318, U13 IXDN614, U14 MAX3485, U15 ISO7320FC, U16 TLV74325, U17 IXDN614, U18 IXDN614, U19 XS-GPC-01, U2 AMC3330, U20 ISO7320FC, U21 IXDN614, U22 TLV74325, U23 LM555xM, U24 LM555xM, U25 LM555xM, U26 LM555xM, U27 LM555xM, U28 MAX3485, U29 MAX3485, U3 IXDN614, U30 MAX3485, U4 ISO7320FC, U5 TLV74325, U6 MAX3485, U7 TLV74325, U8 MAX3485, U9 AD7352

Commit message: development system pcb(s) floorplan
Parts:
- removed J15: Vdc, TerminalBlock_Phoenix:TerminalBlock_Phoenix_MKDS-1,5-2-5.08_1x02_P5.08mm_Horizontal
- removed J18: Vac, TerminalBlock_Phoenix:TerminalBlock_Phoenix_MKDS-1,5-2-5.08_1x02_P5.08mm_Horizontal
- added C64: 220u 450v0v, Capacitor_THT:CP_Radial_D18.0mm_P7.50mm, F.Cu at (162.2, 59.1)
- added C64: 220u 450v0v, Capacitor_THT:CP_Radial_D18.0mm_P7.50mm, F.Cu at (143.1, 39.8)
- added C64: 220u 450v0v, Capacitor_THT:CP_Radial_D18.0mm_P7.50mm, F.Cu at (124.0, 59.2)
- added C64: 220u 450v0v, Capacitor_THT:CP_Radial_D18.0mm_P7.50mm, F.Cu at (162.6, 40.4)
- added C64: 220u 450v0v, Capacitor_THT:CP_Radial_D18.0mm_P7.50mm, F.Cu at (123.7, 40.0)
- added C64: 220u 450v0v, Capacitor_THT:CP_Radial_D18.0mm_P7.50mm, F.Cu at (143.1, 59.4)
- added C64: 220u 450v0v, Capacitor_THT:CP_Radial_D18.0mm_P7.50mm, F.Cu at (181.8, 40.3)
- added C64: 220u 450v0v, Capacitor_THT:CP_Radial_D18.0mm_P7.50mm, F.Cu at (181.7, 59.2)
- added C67: 22n 1000v, Capacitor_THT:C_Rect_L13.0mm_W6.0mm_P10.00mm_FKS3_FKP3_MKS4, B.Cu at (44.6, 55.2)
- added C68: 22n 1000v, Capacitor_THT:C_Rect_L13.0mm_W6.0mm_P10.00mm_FKS3_FKP3_MKS4, B.Cu at (-134.6, 201.8)
- added D6: VBE60-06A, Package_TO_SOT_THT:SOT-227, F.Cu at (55.2, 57.7)
- R5, R6: moved to B.Cu
- moved C38 299.7 mm to (-41.9, 196.7)
- moved C39 299.7 mm to (-41.9, 199.2)
- moved C40 299.7 mm to (-41.9, 201.7)
- moved C41 299.7 mm to (-33.8, 182.4)
- moved C42 299.7 mm to (-41.9, 206.8)
- moved C43 299.7 mm to (-41.9, 209.3)
- moved C44 299.7 mm to (-41.9, 211.8)
- moved C45 299.7 mm to (-41.9, 214.3)
- moved C46 299.7 mm to (-37.9, 196.7)
- moved C47 299.7 mm to (-29.8, 177.4)
- moved C48 299.7 mm to (-37.9, 201.7)
- moved C49 299.7 mm to (-37.9, 204.2)
- moved C50 299.7 mm to (-29.8, 184.9)
- moved C51 299.7 mm to (-29.8, 187.5)
- moved C54 299.7 mm to (-37.9, 211.8)
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Other:
- board size 182.9 x 100.4 mm -> 244.1 x 104.3 mm
- board text added: "DCLINK"
- board text added: "DUMP FET"
