File: pcb/GPC_dev_board.kicad_sch (KiCad schematic)
At the start: 185 parts, among them J1 Conn_01x12, J10 CTRL, J11 Conn_02x06_Top_Bottom, J12 LVIN, J14 Conn_01x04, J15 Vdc, J16 PWMIN, J17 HBRIDGE, J18 Vac, J19 LVIN, J2 Conn_01x12, J20 LVOUT, J3 Conn_02x13_Odd_Even, J4 Conn_02x13_Odd_Even, J5 BATTERY, J6 SECONDARY, J7 3.3V, Q1 IXFN80N50, Q2 IRF4905, Q3 IRF4905, Q4 IRF4905, Q5 IRF4905, Q6 MMBT3904, Q7 MMBT3904, Q8 MMBT3904, Q9 MMBT3904, U1 AMC3330, U10 ISO7320FC, U11 TLV74325, U12 TLV74318, U13 IXDN614, U14 MAX3485, U15 ISO7320FC, U16 TLV74325, U17 IXDN614, U18 IXDN614, U19 XS-GPC-01, U2 AMC3330, U20 ISO7320FC, U21 IXDN614, U22 TLV74325, U23 LM555xM, U24 LM555xM, U25 LM555xM, U26 LM555xM, U27 LM555xM, U28 MAX3485, U29 MAX3485, U3 IXDN614, U30 MAX3485, U4 ISO7320FC, U5 TLV74325, U6 MAX3485, U7 TLV74325, U8 MAX3485, U9 AD7352

Commit message: development system pcb(s) floorplan
Parts:
- removed J15: Vdc, TerminalBlock_Phoenix:TerminalBlock_Phoenix_MKDS-1,5-2-5.08_1x02_P5.08mm_Horizontal, symbol Connector:Screw_Terminal_01x02
- removed J18: Vac, TerminalBlock_Phoenix:TerminalBlock_Phoenix_MKDS-1,5-2-5.08_1x02_P5.08mm_Horizontal, symbol Connector:Screw_Terminal_01x02
- added C63, C64, C65, C66: 220u 450v0v, Capacitor_THT:CP_Radial_D18.0mm_P7.50mm, symbol Device:C_Polarized_Small
- added C67, C68: 22n 1000v, Capacitor_THT:C_Rect_L13.0mm_W6.0mm_P10.00mm_FKS3_FKP3_MKS4, symbol Device:C_Polarized_Small
- added D6: VBE60-06A, Package_TO_SOT_THT:SOT-227, symbol Diode_Bridge:KBPC5008W
Connections:
- new net: C67.1, C67.2
Other:
- note added: "DC Link and Voltage Dividers"
- note removed: "Voltage Dividers"
- moved on the sheet: H15, H16, J20, R1, R2, R3, R4, R5, R6
